File: hardware/pcb/Pointy R1 Flight controller/Pointy R1 Flight controller.kicad_sch (KiCad schematic)
At the start: 0 parts

Commit message: create PCB library env, added main components to sch
Parts:
- added IC1: TEENSY_4.1, footprints:TEENSY41, symbol symbols:TEENSY_4.1
- added LED1: COM-16347, footprints:COM-16347_SPK, symbol symbols:COM-16347
- added LS1: CMI-1295-0585T, footprints:CUI_CMI-1295-0585T, symbol symbols:CMI-1295-0585T
- added Q1, Q2: 2N7002, footprints:SOT95P240X111-3N, symbol symbols:2N7002
- added U1: L7805CV, footprints:TO255P1040X460X1968-3, symbol symbols:L7805CV
- added U2: GY-521, footprints:MODULE_GY-521, symbol symbols:GY-521
